File: LED_Bracelet.kicad_sch (KiCad schematic)
At the start: 46 parts, among them J1 USB-C (Female), J2 LED Strip, J3 LED Filament, Q1 Si2301CDS, SW1 BOOT, U1 TP4056, U2 DW01A-G, U3 FS8205A, U4 TPS61170, U5 SN74AHCT1G125DBVR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

Commit message: Tweaks to the PCB
Parts:
- H1, H2: footprint Custom:Tooling Hole (JLCPCB) -> Custom:JLCPCB ToolingHole
- U7: LCSC (none) -> C51118
Connections:
- net +BATT: now also R14.2
- net GND: no longer R14.2
Other:
- moved on the sheet: R14
Changed lines of the file:
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@@
     (stroke (width 0) (type default))
   )
-  (wire (pts (xy 196.85 52.07) (xy 215.9 52.07))
+  (wire (pts (xy 200.66 52.07) (xy 215.9 52.07))
     (stroke (width 0) (type default))
   )
@@
     )
   )
-  (symbol (lib_id "Device:R_Small") (at 196.85 54.61 0) (unit 1)
-    (in_bom yes) (on_board yes) (dnp no)
-    (property "Reference" "R14" (at 198.12 53.34 0)
-      (effects (font (size 1.27 1.27)) (justify left))
-    )
-    (property "Value" "10k" (at 198.12 55.88 0)
-      (effects (font (size 1.27 1.27)) (justify left))
-    )
-    (property "Footprint" "Resistor_SMD:R_0603_1608Metric" (at 196.85 54.61 0)
-      (effects (font (size 1.27 1.27)) hide)
-    )
-    (property "Datasheet" "~" (at 196.85 54.61 0)
-      (effects (font (size 1.27 1.27)) hide)
-    )
-    (property "LCSC" "C25804" (at 196.85 54.61 0)
+  (symbol (lib_id "Device:R_Small") (at 200.66 49.53 180) (unit 1)
+    (in_bom yes) (on_board yes) (dnp no)
+    (property "Reference" "R14" (at 199.39 50.8 0)
+      (effects (font (size 1.27 1.27)) (justify left))
+    )
+    (property "Value" "10k" (at 199.39 48.26 0)
+      (effects (font (size 1.27 1.27)) (justify left))
+    )
+    (property "Footprint" "Resistor_SMD:R_0603_1608Metric" (at 200.66 49.53 0)
+      (effects (font (size 1.27 1.27)) hide)
+    )
+    (property "Datasheet" "~" (at 200.66 49.53 0)
+      (effects (font (size 1.27 1.27)) hide)
+    )
+    (property "LCSC" "C25804" (at 200.66 49.53 0)
       (effects (font (size 1.27 1.27)) hide)
     )
@@
     )
   )
-  (symbol (lib_id "power:GND") (at 196.85 57.15 0) (unit 1)
-    (in_bom yes) (on_board yes) (dnp no)
-    (property "Reference" "#PWR0114" (at 196.85 63.5 0)
-      (effects (font (size 1.27 1.27)) hide)
-    )
-    (property "Value" "GND" (at 196.85 60.96 0)
-      (effects (font (size 1.27 1.27)))
-    )
-    (property "Footprint" "" (at 196.85 57.15 0)
-      (effects (font (size 1.27 1.27)) hide)
-    )
-    (property "Datasheet" "" (at 196.85 57.15 0)
-      (effects (font (size 1.27 1.27)) hide)
-    )
-    (pin "1")
-    (instances
-      (project "LED_Bracelet"
-        (path "/16a89f0a-88d3-42f5-a8f1-2ef510493fd4"
-          (reference "#PWR0114") (unit 1)
-        )
-      )
-    )
-  )
   (symbol (lib_id "Mechanical:MountingHole_Pad") (at 134.62 182.88 0) (unit 1)
     (in_bom no) (on_board yes) (dnp no)
@@
       (effects (font (size 1.27 1.27)) (justify left) hide)
     )
-    (property "Footprint" "Custom:Tooling Hole (JLCPCB)" (at 160.02 182.88 0)
+    (property "Footprint" "Custom:JLCPCB ToolingHole" (at 160.02 182.88 0)
       (effects (font (size 1.27 1.27)) hide)
     )
     (property "Datasheet" "~" (at 160.02 182.88 0)
+      (effects (font (size 1.27 1.27)) hide)
+    )
+    (property "LCSC" "" (at 160.02 182.88 0)
       (effects (font (size 1.27 1.27)) hide)
     )
@@
     )
     (property "Datasheet" "https://www.diodes.com/assets/Datasheets/AP2112.pdf" (at 36.83 113.03 0)
+      (effects (font (size 1.27 1.27)) hide)
+    )
+    (property "LCSC" "C51118" (at 36.83 115.57 0)
       (effects (font (size 1.27 1.27)) hide)
     )
@@
         (path "/16a89f0a-88d3-42f5-a8f1-2ef510493fd4"
           (reference "R3") (unit 1)
+        )
+      )
+    )
+  )
+  (symbol (lib_id "power:+BATT") (at 200.66 46.99 0) (unit 1)
+    (in_bom yes) (on_board yes) (dnp no)
+    (property "Reference" "#PWR033" (at 200.66 50.8 0)
+      (effects (font (size 1.27 1.27)) hide)
+    )
+    (property "Value" "+BATT" (at 200.66 43.18 0)
+      (effects (font (size 1.27 1.27)))
+    )
+    (property "Footprint" "" (at 200.66 46.99 0)
+      (effects (font (size 1.27 1.27)) hide)
+    )
+    (property "Datasheet" "" (at 200.66 46.99 0)
+      (effects (font (size 1.27 1.27)) hide)
+    )
+    (pin "1")
+    (instances
+      (project "LED_Bracelet"
+        (path "/16a89f0a-88d3-42f5-a8f1-2ef510493fd4"
+          (reference "#PWR033") (unit 1)
         )
       )
@@
       (effects (font (size 1.27 1.27)) (justify left) hide)
     )
-    (property "Footprint" "Custom:Tooling Hole (JLCPCB)" (at 166.37 182.88 0)
+    (property "Footprint" "Custom:JLCPCB ToolingHole" (at 166.37 182.88 0)
       (effects (font (size 1.27 1.27)) hide)
     )
@@
       (effects (font (size 1.27 1.27)) hide)
     )
+    (property "LCSC" "" (at 166.37 182.88 0)
+      (effects (font (size 1.27 1.27)) hide)
+    )

Commit message: First software version + some PCB changes Separate BOOT and Mode buttons. LED Filament MOSFET (Q1) has pulldown resistor and is the correct channel. PlatformIO project + code. Frequently Asked Questions (FAQ).
Parts:
- removed Q1: Si2301CDS, Package_TO_SOT_SMD:SOT-23, symbol PCM_Transistor_MOSFET_AKL:Si2301CDS
- added Q1: AO3400A, Package_TO_SOT_SMD:SOT-23, symbol Transistor_FET:AO3400A
- added R17: 100R, Resistor_SMD:R_0603_1608Metric, symbol Device:R
- added R18: 1k, Resistor_SMD:R_0603_1608Metric, symbol Device:R
- added SW1: Mode, Button_Switch_SMD:Panasonic_EVQPUL_EVQPUC, symbol Switch:SW_Push
- SW2: renamed from SW1; footprint Button_Switch_SMD:Panasonic_EVQPUL_EVQPUC -> Jumper:SolderJumper-2_P1.3mm_Open_RoundedPad1.0x1.5mm
Connections:
- net GND: now also Q1.2 (S), R18.2, SW1.1
- net LED Filament: now also R17.1
- net LED Strip: now also U6.6 (GPIO7); no longer U6.7 (GPIO8)
- net Mode: now reaches U6.15 (GPIO3/ADC1_CH3)
- net Mode: now also SW1.2
- net at J3.1 (Pin_1): now also Q1.3 (D)
- net Strapping 1 renamed Strapping_1
- net Strapping_1: now also U6.7 (GPIO8)
- new net Q1 Gate: Q1.1 (G), R17.2, R18.1
Other:
- note added: "30V 5.7A"
- note removed: "20V 3.1A"
- moved on the sheet: SW2
